File: hardware/alarm-clock.kicad_pcb (KiCad board)
At the start: 2 copper layers, 68.6 x 86.4 mm, 40 parts, among them CON1 BARREL_JACK, CON2 BARREL_JACK, IC1 ATMEGA328P-PU, P1 PROGRAMMER, Q1 Q_NPN_BCE, Q2 Q_NPN_BCE, SW1 SPST, U1 LM7805CT, U2 DS1307, U3 4Dig7Seg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

Commit message: Re-wire to use hardware PWM d'oh
Parts:
- removed REF** (x4): MountingHole_3mm, Mounting_Holes:MountingHole_3mm
- moved R11 117.7 mm to (47.5, 39.1)
- moved R12 117.7 mm to (51.3, 39.1)
- moved C5 116.3 mm to (36.6, 73.4)
- moved C6 116.3 mm to (36.6, 78.5)
- moved D1 116.3 mm to (32.8, 78.5)
- moved D2 116.3 mm to (21.3, 55.6)
- moved U2 116.3 mm to (68.3, 72.8)
- moved BT1 116.3 mm to (75.9, 36.3)
- moved C3 116.3 mm to (22.6, 82.3)
- moved IC1 116.3 mm to (49.3, 54.4)
- moved PB1 116.3 mm to (34.0, 55.6)
- moved PB2 116.3 mm to (72.1, 55.6)
- moved Q2 116.3 mm to (29.0, 64.5)
- moved R1 116.3 mm to (65.8, 92.5)
- moved R2 116.3 mm to (37.8, 64.5)
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Connections:
- Q2 pad 2: GND -> +5V
- R1 pad 1: PC3 -> PB1
- R13 pad 1: PC0 -> PC2
- R14 pad 1: PC1 -> PC3
- R2 pad 1: PC2 -> PB3
- R7 pad 1: PB2 -> PB4
- R9 pad 1: PB3 -> PB5
- U3 pad 10: PB5 -> PC1
- U3 pad 11: PB4 -> PC0
- U3 pad 14: PB1 -> PB2
Routing:
- net GND: track 267.4 -> 1.54 mm, vias 4 -> 0
- net PB1: track 138.5 -> 8.99 mm
- net PB4: track 151.2 -> 75.5 mm, vias 0 -> 2
- net PB2: track 67.7 -> 107.3 mm, vias 0 -> 1
- net PD4: track 37.2 -> 65.8 mm, vias 2 -> 3
- net PB3: track 86.5 -> 64.7 mm, vias 3 -> 4
- net PC0: track 29.0 -> 50.2 mm, vias 1 -> 0
- net PC3: track 37.3 -> 22.5 mm, vias 0 -> 1
- net PC1: track 26.0 -> 38.2 mm, vias 1 -> 0
- net PD2: track 32.9 -> 40.9 mm, vias 1 -> 0
- net PC2: track 18.1 -> 24.4 mm, vias 2 -> 1
- net +5V: track 141.7 -> 147.3 mm, vias 2 -> 3
- net PB5: track 74.3 -> 69.0 mm, vias 2 -> 4
- net Net-(R14-Pad2): track 11.7 -> 7.07 mm
- net Net-(R6-Pad1): track 15.9 -> 11.7 mm
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
Commit message: WIP on V3
Parts:
- BT1, Q2, R1, R10, R11, R12, R13, R14, R2, R3, R4, R5, R6, R7, R8, R9: moved to F.Cu
- C1: footprint Capacitors_ThroughHole:C_Radial_D6.3_L11.2_P2.5 -> Capacitors_THT:CP_Radial_D6.3mm_P2.50mm
- C3: footprint Capacitors_ThroughHole:C_Radial_D5_L11_P2 -> Capacitors_THT:CP_Radial_D5.0mm_P2.00mm
- C5, C6: footprint Capacitors_ThroughHole:C_Disc_D3_P2.5 -> Capacitors_SMD:C_1210_HandSoldering
- D1: footprint Diodes_THT:Diode_DO-41_SOD81_Horizontal_RM10 -> Diodes_THT:D_DO-41_SOD81_P10.16mm_Horizontal
- IC1: footprint Housings_DIP:DIP-28_W7.62mm_Socket -> Housings_QFP:TQFP-32_7x7mm_Pitch0.8mm
- Y1: footprint Crystals:Crystal_Round_Horizontal_2mm -> Crystals:Crystal_Round_d2.0mm_Vertical
- moved SW1 166.2 mm to (181.5, 95.0), turned to 0 degrees
- moved R5 162.0 mm to (181.5, 95.0), turned to 0 degrees
- moved R7 159.1 mm to (181.5, 95.0), turned to 0 degrees
- moved R6 155.8 mm to (181.5, 95.0), turned to 0 degrees
- moved Q2 155.6 mm to (181.5, 95.0), turned to 0 degrees
- moved R8 152.3 mm to (181.5, 95.0), turned to 0 degrees
- moved R10 148.7 mm to (181.5, 95.0), turned to 0 degrees
- moved R2 146.9 mm to (181.5, 95.0), turned to 0 degrees
- moved C5 146.5 mm to (181.5, 95.0)
- moved C6 145.9 mm to (181.5, 95.0)
- moved R11 145.2 mm to (181.5, 95.0), turned to 0 degrees
- moved R12 141.7 mm to (181.5, 95.0), turned to 0 degrees
- moved SP1 138.9 mm to (164.0, 89.0), turned to 0 degrees
- moved R9 138.2 mm to (181.5, 95.0), turned to 0 degrees
- moved R13 134.7 mm to (181.5, 95.0), turned to 0 degrees
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Connections:
- IC1 pad 21: (no net) -> Net-(IC1-Pad21)
- U2 pad 7: (no net) -> Net-(U2-Pad7)
Routing:
- net +5V: track 147.3 -> 0.00 mm, vias 3 -> 0
- net PB2: track 107.3 -> 0.00 mm, vias 1 -> 0
- net PB4: track 75.5 -> 0.00 mm, vias 2 -> 0
- net PB5: track 69.0 -> 0.00 mm, vias 4 -> 0
- net PD4: track 65.8 -> 0.00 mm, vias 3 -> 0
- net PB3: track 64.7 -> 0.00 mm, vias 4 -> 0
- net VPP: track 58.6 -> 0.00 mm
- net PB0: track 55.7 -> 0.00 mm, vias 2 -> 0
- net PD7: track 51.6 -> 0.00 mm, vias 2 -> 0
- net PC0: track 50.2 -> 0.00 mm
- net PD6: track 47.6 -> 0.00 mm, vias 2 -> 0
- net RESET: track 45.1 -> 0.00 mm, vias 1 -> 0
- net PD5: track 45.0 -> 0.00 mm, vias 2 -> 0
- net PD2: track 40.9 -> 0.00 mm
- net PC1: track 38.2 -> 0.00 mm
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- removed copper zone on B.Cu, net GND
- removed copper zone on F.Cu, net GND
Other:
- board outline removed
- board text removed: "↑ TIME ALARM"
- board text removed: "↓ TIME ALARM"

Commit message: WIP V3
Parts:
- removed C5, C6: 20pF, Capacitors_SMD:C_1210_HandSoldering
- removed IC1: ATMEGA328P-PU, Housings_QFP:TQFP-32_7x7mm_Pitch0.8mm
- removed R10, R11, R12, R13, R14, R6, R7, R8, R9: 2.2k, Resistors_SMD:R_1210_HandSoldering
- removed Y2: 16MHz, Crystals:Crystal_HC49-U_Vertical
- added C2: 1µF, Capacitors_SMD:C_1206_HandSoldering, F.Cu at (51.0, 123.5)
- added C4: 20pF, Capacitors_SMD:C_1206_HandSoldering, B.Cu at (83.0, 90.0)
- added J1: CONN_01X04, Pin_Headers:Pin_Header_Straight_1x04_Pitch2.54mm, B.Cu at (67.5, 142.5)
- added PB3: push_button, custom:KS_BUTTON, F.Cu at (50.0, 137.0)
- added REF**: MountingHole_2.7mm_M2.5_ISO7380_Pad, Mounting_Holes:MountingHole_2.7mm_M2.5_ISO7380_Pad, F.Cu at (87.0, 88.0)
- added REF**: MountingHole_2.7mm_M2.5_ISO7380_Pad, Mounting_Holes:MountingHole_2.7mm_M2.5_ISO7380_Pad, F.Cu at (87.0, 142.0)
- added REF**: MountingHole_2.7mm_M2.5_ISO7380_Pad, Mounting_Holes:MountingHole_2.7mm_M2.5_ISO7380_Pad, F.Cu at (43.0, 142.0)
- added REF**: MountingHole_2.7mm_M2.5_ISO7380_Pad, Mounting_Holes:MountingHole_2.7mm_M2.5_ISO7380_Pad, F.Cu at (43.0, 88.0)
- BT1, CON1, CON2: moved to B.Cu
- C1: footprint Capacitors_THT:CP_Radial_D6.3mm_P2.50mm -> Capacitors_SMD:C_1206_HandSoldering
- C3: value 1µF -> 20pF; footprint Capacitors_THT:CP_Radial_D5.0mm_P2.00mm -> Capacitors_SMD:C_1206_HandSoldering; moved to B.Cu
- D1: footprint Diodes_THT:D_DO-41_SOD81_P10.16mm_Horizontal -> Diodes_SMD:D_1206; moved to B.Cu
- D2: footprint LEDs:LED_D5.0mm -> LEDs:LED_1206
- PB1, PB2: footprint Buttons_Switches_THT:SW_PUSH-12mm -> custom:KS_BUTTON
- Q1: moved to F.Cu
- R1, R2: value 3.3k -> 3k3; footprint Resistors_SMD:R_1210_HandSoldering -> Resistors_SMD:R_1206_HandSoldering
- R3: value 2.2k -> 2k2; footprint Resistors_SMD:R_1210_HandSoldering -> Resistors_SMD:R_1206_HandSoldering; moved to B.Cu
- R4: value 2.2k -> 2k2; footprint Resistors_SMD:R_1210_HandSoldering -> Resistors_SMD:R_1206_HandSoldering
- R5: value 270 -> 2k2; footprint Resistors_SMD:R_1210_HandSoldering -> Resistors_SMD:R_1206_HandSoldering
- U1: footprint Power_Integrations:TO-220 -> TO_SOT_Packages_THT:TO-220_Horizontal; moved to B.Cu
- U2: value DS1307 -> DS3232; footprint Housings_DIP:DIP-8_W7.62mm_LongPads -> Housings_SOIC:SOIC-20W_7.5x12.8mm_Pitch1.27mm
- U3: value 4Dig7Seg -> ATMEGA328-AU; footprint custom:4Dig7Seg -> Housings_QFP:TQFP-32_7x7mm_Pitch0.8mm
- Y1: value 38.7kHz -> 16MHz; footprint Crystals:Crystal_Round_d2.0mm_Vertical -> Crystals:Crystal_HC49-U_Vertical
- moved R3 143.3 mm to (42.5, 130.0), turned to 270 degrees
- moved Q2 133.6 mm to (48.0, 100.0), turned to 90 degrees
- moved Q1 131.2 mm to (51.2, 111.0), turned to 270 degrees
- moved R2 126.6 mm to (55.0, 101.0), turned to 180 degrees
- moved SP1 120.2 mm to (44.0, 96.0)
- moved CON2 117.5 mm to (48.0, 121.0)
- moved R4 111.7 mm to (70.0, 102.0), turned to 90 degrees
- moved R1 110.2 mm to (72.0, 107.0), turned to 180 degrees
- moved R5 108.7 mm to (73.0, 102.0), turned to 90 degrees
- moved D2 102.8 mm to (42.5, 130.0), turned to 270 degrees
- moved SW1 101.9 mm to (87.0, 133.0), turned to 270 degrees
- moved P1 97.3 mm to (62.5, 92.5), turned to 90 degrees
- moved PB2 93.4 mm to (76.0, 137.0)
- moved C1 88.0 mm to (51.0, 118.5)
- moved D1 79.5 mm to (57.0, 116.5), turned to 90 degrees
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Connections:
- C3 pad 1: +5V -> GND
- C3 pad 2: GND -> Net-(C3-Pad2)
- R3 pad 2: PC4 -> Net-(D2-Pad2)
- R4 pad 2: PC5 -> SCL
- R5 pad 2: Net-(D2-Pad2) -> SDA
- SW1 pad 1: PD2 -> PD3
- U2 pad 1: Net-(U2-Pad1) -> GND
- U2 pad 2: Net-(U2-Pad2) -> GND
- U2 pad 3: Net-(BT1-Pad1) -> (no net)
- U2 pad 4: GND -> +5V
- U2 pad 5: PC4 -> (no net)
- U2 pad 6: PC5 -> (no net)
- U2 pad 7: Net-(U2-Pad7) -> GND
- U2 pad 8: +5V -> GND
- U3 pad 1: Net-(R6-Pad1) -> PD3
- U3 pad 10: PC1 -> (no net)
- U3 pad 11: PC0 -> (no net)
- U3 pad 12: Net-(R9-Pad2) -> (no net)
- U3 pad 13: Net-(R7-Pad2) -> PB1
- U3 pad 14: PB2 -> (no net)
- U3 pad 2: Net-(R8-Pad1) -> (no net)
- U3 pad 3: Net-(R10-Pad1) -> GND
- U3 pad 4: Net-(R11-Pad1) -> +5V
- U3 pad 5: Net-(R12-Pad1) -> GND
- U3 pad 6: PD3 -> (no net)
- U3 pad 7: GND -> Net-(C3-Pad2)
- U3 pad 8: Net-(R14-Pad2) -> Net-(C4-Pad2)
- U3 pad 9: Net-(R13-Pad2) -> (no net)
- Y1 pad 1: Net-(U2-Pad2) -> Net-(C4-Pad2)
- Y1 pad 2: Net-(U2-Pad1) -> Net-(C3-Pad2)
Other:
- board outline added: 50 x 60 mm
- board text added: "▲"
- board text added: "▼"
