File: hardware/alarm-clock.sch (KiCad schematic (older format))
At the start: 33 parts, among them CON1 BARREL_JACK, CON2 BARREL_JACK, IC1 ATMEGA328-P, Q1 Q_NPN_BCE, SW1 SWITCH_INV, SW2 SW_PUSH, SW3 SW_PUSH, U1 LM7805CT, U2 DS1307, U3 4Dig7Seg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

Commit message: Update schematic
Parts:
- added C4: 12.5pF, Capacitors_ThroughHole:C_Disc_D3_P2.5, symbol C_Small
- added C?: C_Small, symbol C_Small
- renumbered C2 to C3, C3 to C5, C4 to C6
Connections:
- net GND: now also C4.1, C?.1
- net at U2.2 (X2), Y1.1: now also C?.2
- net at U2.1 (X1), Y1.2: now also C4.2
Changed lines of the file:
@@
 $EndComp
 $Comp
-L CP1_Small C2
+L CP1_Small C3
 U 1 1 580D3FDC
 P 1600 3150
-F 0 "C2" H 1610 3220 50  0000 L CNN
+F 0 "C3" H 1610 3220 50  0000 L CNN
 F 1 "1µF" H 1610 3070 50  0000 L CNN
 F 2 "Capacitors_ThroughHole:C_Radial_D6.3_L11.2_P2.5" H 1600 3150 50  0001 C CNN
@@
 PC2
 $Comp
-L C_Small C3
+L C_Small C5
 U 1 1 580DB46E
 P 4700 1500
-F 0 "C3" H 4710 1570 50  0000 L CNN
+F 0 "C5" H 4710 1570 50  0000 L CNN
 F 1 "20pF" H 4710 1420 50  0000 L CNN
 F 2 "Capacitors_ThroughHole:C_Disc_D3_P2.5" H 4700 1500 50  0001 C CNN
@@
 $EndComp
 $Comp
-L C_Small C4
+L C_Small C6
 U 1 1 580DB5B3
 P 4700 1900
-F 0 "C4" H 4710 1970 50  0000 L CNN
+F 0 "C6" H 4710 1970 50  0000 L CNN
 F 1 "20pF" H 4710 1820 50  0000 L CNN
 F 2 "Capacitors_ThroughHole:C_Disc_D3_P2.5" H 4700 1900 50  0001 C CNN
@@
 	1650 5800 1750 5800
 Wire Wire Line
-	1750 5900 1400 5900
-Wire Wire Line
-	1400 5900 1400 5800
-Wire Wire Line
-	1400 5800 1450 5800
+	1350 5900 1750 5900
+Wire Wire Line
+	1350 5550 1350 5900
+Wire Wire Line
+	1350 5800 1450 5800
 Wire Wire Line
 	1250 4500 1500 4500
@@
 Text GLabel 4000 3050 2    60   Input ~ 0
 PD4
+$Comp
+L C_Small C?
+U 1 1 5823D955
+P 1350 5450
+F 0 "C?" H 1360 5520 50  0000 L CNN
+F 1 "C_Small" H 1360 5370 50  0000 L CNN
+F 2 "" H 1350 5450 50  0000 C CNN
+F 3 "" H 1350 5450 50  0000 C CNN
+	1    1350 5450
+	1    0    0    -1
+$EndComp
+$Comp
+L C_Small C4
+U 1 1 5823D9D7
+P 1700 5450
+F 0 "C4" H 1710 5520 50  0000 L CNN
+F 1 "12.5pF" H 1710 5370 50  0000 L CNN
+F 2 "Capacitors_ThroughHole:C_Disc_D3_P2.5" H 1700 5450 50  0001 C CNN
+F 3 "" H 1700 5450 50  0000 C CNN
+	1    1700 5450
+	1    0    0    -1
+$EndComp
+Connection ~ 1350 5800
+Wire Wire Line
+	1700 5800 1700 5550
+Connection ~ 1700 5800
+Wire Wire Line
+	1350 5350 1350 5250
+Wire Wire Line
+	950  5250 1700 5250
+Wire Wire Line
+	1700 5250 1700 5350
+Wire Wire Line
+	950  5250 950  5350
+Connection ~ 1350 5250
+$Comp
+L GND #PWR027
+U 1 1 5823DC58
+P 950 5350
+F 0 "#PWR027" H 950 5100 50  0001 C CNN
+F 1 "GND" H 950 5200 50  0000 C CNN
+F 2 "" H 950 5350 50  0000 C CNN
+F 3 "" H 950 5350 50  0000 C CNN
+	1    950  5350
+	1    0    0    -1
+$EndComp
 $EndSCHEMATC

Commit message: Updated schematic w/ SMD and working buzzer
Parts:
- added Q2: Q_NPN_BCE, TO_SOT_Packages_SMD:SOT-23_Handsoldering, symbol Q_NPN_BCE
- added R2: 3.3k, Resistors_SMD:R_1210_HandSoldering, symbol R
- BT1: footprint custom:CR2032 -> custom:bat_holder_20mm_smd
- C1: footprint Capacitors_ThroughHole:C_Radial_D5_L11_P2 -> Capacitors_ThroughHole:C_Radial_D6.3_L11.2_P2.5
- C2: renamed from C?; value C_Small -> 12.5pF; footprint (none) -> Capacitors_ThroughHole:C_Disc_D3_P2.5
- C3: footprint Capacitors_ThroughHole:C_Radial_D6.3_L11.2_P2.5 -> Capacitors_ThroughHole:C_Radial_D5_L11_P2
- Q1: footprint TO_SOT_Packages_THT:TO-92_Inline_Narrow_Oval -> TO_SOT_Packages_SMD:SOT-23_Handsoldering
- R1: footprint Resistors_ThroughHole:Resistor_Horizontal_RM7mm -> Resistors_SMD:R_1210_HandSoldering
- R10: renamed from R9; footprint Resistors_ThroughHole:Resistor_Horizontal_RM7mm -> Resistors_SMD:R_1210_HandSoldering
- R11: renamed from R10; footprint Resistors_ThroughHole:Resistor_Horizontal_RM7mm -> Resistors_SMD:R_1210_HandSoldering
- R12: renamed from R11; footprint Resistors_ThroughHole:Resistor_Horizontal_RM7mm -> Resistors_SMD:R_1210_HandSoldering
- R13: renamed from R12; footprint Resistors_ThroughHole:Resistor_Horizontal_RM7mm -> Resistors_SMD:R_1210_HandSoldering
- R14: renamed from R13; footprint Resistors_ThroughHole:Resistor_Horizontal_RM7mm -> Resistors_SMD:R_1210_HandSoldering
- R3: renamed from R2; footprint Resistors_ThroughHole:Resistor_Horizontal_RM7mm -> Resistors_SMD:R_1210_HandSoldering
- R4: renamed from R3; footprint Resistors_ThroughHole:Resistor_Horizontal_RM7mm -> Resistors_SMD:R_1210_HandSoldering
- R5: renamed from R4; footprint Resistors_ThroughHole:Resistor_Horizontal_RM7mm -> Resistors_SMD:R_1210_HandSoldering
- R6: renamed from R5; footprint Resistors_ThroughHole:Resistor_Horizontal_RM7mm -> Resistors_SMD:R_1210_HandSoldering
- R7: renamed from R6; footprint Resistors_ThroughHole:Resistor_Horizontal_RM7mm -> Resistors_SMD:R_1210_HandSoldering
- R8: renamed from R7; footprint Resistors_ThroughHole:Resistor_Horizontal_RM7mm -> Resistors_SMD:R_1210_HandSoldering
- R9: renamed from R8; footprint Resistors_ThroughHole:Resistor_Horizontal_RM7mm -> Resistors_SMD:R_1210_HandSoldering
- Y1: footprint Crystals:Crystal_Round_Vertical_2mm -> Crystals:Crystal_Round_Horizontal_2mm
Connections:
- net +5V: now also IC1.1 ((PCINT14/~RESET~)PC6), IC1.20 (AVCC)
- net GND: now also Q2.2 (C)
- net PC2: now also R2.1; no longer SP1.1
- new net: Q2.3 (E), SP1.1
- new net: Q2.1 (B), R2.2
- no-connect marks 4 -> 2
Other:
- moved on the sheet: SP1, SW2, SW3

Commit message: Cleanup and update some footprints
Parts:
- removed C2, C4: 12.5pF, Capacitors_ThroughHole:C_Disc_D3_P2.5, symbol C_Small
- BT1: symbol Battery -> Battery-RESCUE-alarm-clock
- D2: symbol LED -> LED-RESCUE-alarm-clock
- Y2: footprint Crystals:Crystal_HC50-U_Vertical -> Crystals:Crystal_HC49-U_Vertical
Connections:
- wire segments 62 -> 57
Changed lines of the file:
@@
 EESchema Schematic File Version 2
+LIBS:alarm-clock-rescue
 LIBS:power
 LIBS:device
@@
 F 0 "Y2" H 4450 1800 50  0000 C CNN
 F 1 "16MHz" H 4450 1600 50  0000 C CNN
-F 2 "Crystals:Crystal_HC50-U_Vertical" H 4450 1700 50  0001 C CNN
+F 2 "Crystals:Crystal_HC49-U_Vertical" H 4450 1700 50  0001 C CNN
 F 3 "" H 4450 1700 50  0000 C CNN
 	1    4450 1700
@@
 PC4
 $Comp
-L Battery BT1
+L Battery-RESCUE-alarm-clock BT1
 U 1 1 580D4C5B
 P 1250 6150
@@
 	1350 5900 1750 5900
 Wire Wire Line
-	1350 5550 1350 5900
+	1350 5800 1350 5900
 Wire Wire Line
 	1350 5800 1450 5800
@@
 $EndComp
 $Comp
-L LED D2
+L LED-RESCUE-alarm-clock D2
 U 1 1 58220B55
 P 4700 5650
@@
 Text GLabel 4000 3050 2    60   Input ~ 0
 PD4
-$Comp
-L C_Small C2
-U 1 1 5823D955
-P 1350 5450
-F 0 "C2" H 1360 5520 50  0000 L CNN
-F 1 "12.5pF" H 1360 5370 50  0000 L CNN
-F 2 "Capacitors_ThroughHole:C_Disc_D3_P2.5" H 1350 5450 50  0001 C CNN
-F 3 "" H 1350 5450 50  0000 C CNN
-	1    1350 5450
-	1    0    0    -1
-$EndComp
-$Comp
-L C_Small C4
-U 1 1 5823D9D7
-P 1700 5450
-F 0 "C4" H 1710 5520 50  0000 L CNN
-F 1 "12.5pF" H 1710 5370 50  0000 L CNN
-F 2 "Capacitors_ThroughHole:C_Disc_D3_P2.5" H 1700 5450 50  0001 C CNN
-F 3 "" H 1700 5450 50  0000 C CNN
-	1    1700 5450
-	1    0    0    -1
-$EndComp
 Connection ~ 1350 5800
-Wire Wire Line
-	1700 5800 1700 5550
 Connection ~ 1700 5800
-Wire Wire Line
-	1350 5350 1350 5250
-Wire Wire Line
-	950  5250 1700 5250
-Wire Wire Line
-	1700 5250 1700 5350
-Wire Wire Line
-	950  5250 950  5350
-Connection ~ 1350 5250
-$Comp
-L GND #PWR027
-U 1 1 5823DC58
-P 950 5350
-F 0 "#PWR027" H 950 5100 50  0001 C CNN
-F 1 "GND" H 950 5200 50  0000 C CNN
-F 2 "" H 950 5350 50  0000 C CNN
-F 3 "" H 950 5350 50  0000 C CNN
-	1    950  5350
-	1    0    0    -1
-$EndComp
 $Comp
 L Q_NPN_BCE Q2
@@
 	3000 4350 3200 4350
 $Comp
-L GND #PWR028
+L GND #PWR027
 U 1 1 585ABDB0
 P 2450 4350
-F 0 "#PWR028" H 2450 4100 50  0001 C CNN
+F 0 "#PWR027" H 2450 4100 50  0001 C CNN
 F 1 "GND" H 2450 4200 50  0000 C CNN
 F 2 "" H 2450 4350 50  0000 C CNN
@@
 	2600 4350 2450 4350
 $Comp
-L +5V #PWR029
+L +5V #PWR028
 U 1 1 585AC913
 P 4400 2500
-F 0 "#PWR029" H 4400 2350 50  0001 C CNN
+F 0 "#PWR028" H 4400 2350 50  0001 C CNN
 F 1 "+5V" H 4400 2640 50  0000 C CNN
 F 2 "" H 4400 2500 50  0000 C CNN
@@
 	4000 2500 4400 2500
 $Comp
-L +5V #PWR030
+L +5V #PWR029
 U 1 1 585ACDE6
 P 2100 1350
-F 0 "#PWR030" H 2100 1200 50  0001 C CNN
+F 0 "#PWR029" H 2100 1200 50  0001 C CNN
 F 1 "+5V" H 2100 1490 50  0000 C CNN
 F 2 "" H 2100 1350 50  0000 C CNN

Commit message: WIP Cleaning up schematic
Parts:
- removed BT1: 3V, custom:bat_holder_20mm_smd, symbol Battery-RESCUE-alarm-clock
- removed D2: LED, LEDs:LED-5MM, symbol LED-RESCUE-alarm-clock
- removed IC1: ATMEGA328-P, Housings_DIP:DIP-28_W7.62mm, symbol ATMEGA328-P
- removed SW1: SWITCH_INV, Buttons_Switches_THT:SW_Micro_SPST, symbol SWITCH_INV
- removed SW2, SW3: SW_PUSH, Buttons_Switches_ThroughHole:SW_PUSH-12mm, symbol SW_PUSH
- added BT1: 3V, symbol Battery_Cell
- added D2: LED, symbol LED
- added IC1: ATMEGA328P-PU, DIL28, symbol ATMEGA328P-PU
- added PB1, PB2: push_button, symbol push_button
- added SW1: SPST, symbol SPST
- SP1: symbol SPEAKER -> Speaker
Connections:
- wire segments 57 -> 58

Commit message: Add programmer port
Parts:
- added P1: PROGRAMMER, Pin_Headers:Pin_Header_Straight_2x03_Pitch2.54mm, symbol CONN_02X03
- BT1: footprint (none) -> custom:CR2032_SMD
- CON1, CON2: footprint Connectors:BARREL_JACK -> custom:BARREL_JACK
- D2: footprint (none) -> LEDs:LED_D5.0mm
- IC1: footprint DIL28 -> Housings_DIP:DIP-28_W7.62mm_Socket
- PB1, PB2: footprint (none) -> Buttons_Switches_THT:SW_PUSH-12mm
- SW1: footprint (none) -> Buttons_Switches_THT:SW_Micro_SPST
Connections:
- net labels added: RESET
- wire segments 58 -> 57
Changed lines of the file:
@@
 PC4
 $Comp
-L GND #PWR7
+L GND #PWR01
 U 1 1 580D4D32
 P 1250 6300
-F 0 "#PWR7" H 1250 6050 50  0001 C CNN
+F 0 "#PWR01" H 1250 6050 50  0001 C CNN
 F 1 "GND" H 1250 6150 50  0000 C CNN
 F 2 "" H 1250 6300 50  0000 C CNN
@@
 $EndComp
 $Comp
-L GND #PWR9
+L GND #PWR02
 U 1 1 580D4F57
 P 1750 6100
-F 0 "#PWR9" H 1750 5850 50  0001 C CNN
+F 0 "#PWR02" H 1750 5850 50  0001 C CNN
 F 1 "GND" H 1750 5950 50  0000 C CNN
 F 2 "" H 1750 6100 50  0000 C CNN
@@
 $EndComp
 $Comp
-L GND #PWR15
+L GND #PWR03
 U 1 1 580D5051
 P 2100 3350
-F 0 "#PWR15" H 2100 3100 50  0001 C CNN
+F 0 "#PWR03" H 2100 3100 50  0001 C CNN
 F 1 "GND" H 2100 3200 50  0000 C CNN
 F 2 "" H 2100 3350 50  0000 C CNN
@@
 $EndComp
 $Comp
-L GND #PWR8
+L GND #PWR04
 U 1 1 580D5134
 P 1400 3250
-F 0 "#PWR8" H 1400 3000 50  0001 C CNN
+F 0 "#PWR04" H 1400 3000 50  0001 C CNN
 F 1 "GND" H 1400 3100 50  0000 C CNN
 F 2 "" H 1400 3250 50  0000 C CNN
@@
 $EndComp
 $Comp
-L GND #PWR23
+L GND #PWR05
 U 1 1 580D51A4
 P 5000 1700
-F 0 "#PWR23" H 5000 1450 50  0001 C CNN
+F 0 "#PWR05" H 5000 1450 50  0001 C CNN
 F 1 "GND" H 5000 1550 50  0000 C CNN
 F 2 "" H 5000 1700 50  0000 C CNN
@@
 $EndComp
 $Comp
-L GND #PWR25
+L GND #PWR06
 U 1 1 580D567E
 P 5000 4900
-F 0 "#PWR25" H 5000 4650 50  0001 C CNN
+F 0 "#PWR06" H 5000 4650 50  0001 C CNN
 F 1 "GND" H 5000 4750 50  0000 C CNN
 F 2 "" H 5000 4900 50  0000 C CNN
@@
 $EndComp
 $Comp
-L GND #PWR24
+L GND #PWR07
 U 1 1 580D56DD
 P 5000 4450
-F 0 "#PWR24" H 5000 4200 50  0001 C CNN
+F 0 "#PWR07" H 5000 4200 50  0001 C CNN
 F 1 "GND" H 5000 4300 50  0000 C CNN
 F 2 "" H 5000 4450 50  0000 C CNN
@@
 $EndComp
 $Comp
-L GND #PWR11
+L GND #PWR08
 U 1 1 580D5E88
 P 2000 4500
-F 0 "#PWR11" H 2000 4250 50  0001 C CNN
+F 0 "#PWR08" H 2000 4250 50  0001 C CNN
 F 1 "GND" H 2000 4350 50  0000 C CNN
 F 2 "" H 2000 4500 50  0000 C CNN
@@
 PC1
 $Comp
-L GND #PWR21
+L GND #PWR09
 U 1 1 580DA773
 P 3950 5550
-F 0 "#PWR21" H 3950 5300 50  0001 C CNN
+F 0 "#PWR09" H 3950 5300 50  0001 C CNN
 F 1 "GND" H 3950 5400 50  0000 C CNN
 F 2 "" H 3950 5550 50  0000 C CNN
@@
 $EndComp
 $Comp
-L GND #PWR20
+L GND #PWR010
 U 1 1 580DAD7E
 P 3050 4450
-F 0 "#PWR20" H 3050 4200 50  0001 C CNN
+F 0 "#PWR010" H 3050 4200 50  0001 C CNN
 F 1 "GND" H 3050 4300 50  0000 C CNN
 F 2 "" H 3050 4450 50  0000 C CNN
@@
 $EndComp
 $Comp
-L +5V #PWR17
+L +5V #PWR011
 U 1 1 580DD982
 P 2650 5800
-F 0 "#PWR17" H 2650 5650 50  0001 C CNN
+F 0 "#PWR011" H 2650 5650 50  0001 C CNN
 F 1 "+5V" H 2650 5940 50  0000 C CNN
 F 2 "" H 2650 5800 50  0000 C CNN
@@
 $EndComp
 $Comp
-L +5V #PWR18
+L +5V #PWR012
 U 1 1 580DDA0B
 P 2800 5550
-F 0 "#PWR18" H 2800 5400 50  0001 C CNN
+F 0 "#PWR012" H 2800 5400 50  0001 C CNN
 F 1 "+5V" H 2800 5690 50  0000 C CNN
 F 2 "" H 2800 5550 50  0000 C CNN
@@
 $EndComp
 $Comp
-L +5V #PWR19
+L +5V #PWR013
 U 1 1 580DDA94
 P 3000 5550
-F 0 "#PWR19" H 3000 5400 50  0001 C CNN
+F 0 "#PWR013" H 3000 5400 50  0001 C CNN
 F 1 "+5V" H 3000 5690 50  0000 C CNN
 F 2 "" H 3000 5550 50  0000 C CNN
@@
 $EndComp
 $Comp
-L +5V #PWR10
+L +5V #PWR014
 U 1 1 580DF563
 P 1950 2700
-F 0 "#PWR10" H 1950 2550 50  0001 C CNN
+F 0 "#PWR014" H 1950 2550 50  0001 C CNN
 F 1 "+5V" H 1950 2840 50  0000 C CNN
 F 2 "" H 1950 2700 50  0000 C CNN
@@
 $EndComp
 $Comp
-L +5V #PWR12
+L +5V #PWR015
 U 1 1 580DF644
 P 2100 1050
-F 0 "#PWR12" H 2100 900 50  0001 C CNN
+F 0 "#PWR015" H 2100 900 50  0001 C CNN
 F 1 "+5V" H 2100 1190 50  0000 C CNN
 F 2 "" H 2100 1050 50  0000 C CNN
@@
 $EndComp
 $Comp
-L GND #PWR14
+L GND #PWR016
 U 1 1 580DF8BC
 P 2100 3250
-F 0 "#PWR14" H 2100 3000 50  0001 C CNN
+F 0 "#PWR016" H 2100 3000 50  0001 C CNN
 F 1 "GND" H 2100 3100 50  0000 C CNN
 F 2 "" H 2100 3250 50  0000 C CNN
@@
 $EndComp
 $Comp
-L VPP #PWR3
+L VPP #PWR017
 U 1 1 580E043A
 P 850 2700
-F 0 "#PWR3" H 850 2550 50  0001 C CNN
+F 0 "#PWR017" H 850 2550 50  0001 C CNN
 F 1 "VPP" H 850 2850 50  0000 C CNN
 F 2 "" H 850 2700 50  0000 C CNN
@@
 $EndComp
 $Comp
-L PWR_FLAG #FLG1
+L PWR_FLAG #FLG018
 U 1 1 581E8BD4
 P 950 700
-F 0 "#FLG1" H 950 795 50  0001 C CNN
+F 0 "#FLG018" H 950 795 50  0001 C CNN
 F 1 "PWR_FLAG" H 950 880 50  0000 C CNN
 F 2 "" H 950 700 50  0000 C CNN
@@
 $EndComp
 $Comp
-L PWR_FLAG #FLG2
+L PWR_FLAG #FLG019
 U 1 1 581E8CBA
 P 950 950
-F 0 "#FLG2" H 950 1045 50  0001 C CNN
+F 0 "#FLG019" H 950 1045 50  0001 C CNN
 F 1 "PWR_FLAG" H 950 1130 50  0000 C CNN
 F 2 "" H 950 950 50  0000 C CNN
@@
 $EndComp
 $Comp
-L GND #PWR2
+L GND #PWR020
 U 1 1 581E8FC3
 P 650 950
-F 0 "#PWR2" H 650 700 50  0001 C CNN
+F 0 "#PWR020" H 650 700 50  0001 C CNN
 F 1 "GND" H 650 800 50  0000 C CNN
 F 2 "" H 650 950 50  0000 C CNN
@@
 $EndComp
 $Comp
-L VPP #PWR1
+L VPP #PWR021
 U 1 1 581E97E3
 P 650 700
-F 0 "#PWR1" H 650 550 50  0001 C CNN
+F 0 "#PWR021" H 650 550 50  0001 C CNN
 F 1 "VPP" H 650 850 50  0000 C CNN
 F 2 "" H 650 700 50  0000 C CNN
@@
 	5750 3700 5750 3450
 $Comp
-L GND #PWR27
+L GND #PWR022
 U 1 1 581FB1F9
 P 6250 3450
-F 0 "#PWR27" H 6250 3200 50  0001 C CNN
+F 0 "#PWR022" H 6250 3200 50  0001 C CNN
 F 1 "GND" H 6250 3300 50  0000 C CNN
 F 2 "" H 6250 3450 50  0000 C CNN
@@
 F 0 "CON1" H 950 4000 50  0000 C CNN
 F 1 "BARREL_JACK" H 950 3550 50  0000 C CNN
-F 2 "Connectors:BARREL_JACK" H 950 3750 50  0001 C CNN
+F 2 "custom:BARREL_JACK" H 950 3750 50  0001 C CNN
 F 3 "" H 950 3750 50  0000 C CNN
 	1    950  3750
@@
 F 0 "CON2" H 950 4750 50  0000 C CNN
 F 1 "BARREL_JACK" H 950 4300 50  0000 C CNN
-F 2 "Connectors:BARREL_JACK" H 950 4500 50  0001 C CNN
+F 2 "custom:BARREL_JACK" H 950 4500 50  0001 C CNN
 F 3 "" H 950 4500 50  0000 C CNN
 	1    950  4500
@@
 $EndComp
 $Comp
-L VPP #PWR6
+L VPP #PWR023
 U 1 1 58203612
 P 1250 4400
-F 0 "#PWR6" H 1250 4250 50  0001 C CNN
+F 0 "#PWR023" H 1250 4250 50  0001 C CNN
 F 1 "VPP" H 1250 4550 50  0000 C CNN
 F 2 "" H 1250 4400 50  0000 C CNN
@@
 $EndComp
 $Comp
-L GND #PWR5
+L GND #PWR024
 U 1 1 582036C2
 P 1250 3850
-F 0 "#PWR5" H 1250 3600 50  0001 C CNN
+F 0 "#PWR024" H 1250 3600 50  0001 C CNN
 F 1 "GND" H 1250 3700 50  0000 C CNN
 F 2 "" H 1250 3850 50  0000 C CNN
@@
 $EndComp
 $Comp
-L VPP #PWR4
+L VPP #PWR025
 U 1 1 58203748
 P 1250 3650
-F 0 "#PWR4" H 1250 3500 50  0001 C CNN
+F 0 "#PWR025" H 1250 3500 50  0001 C CNN
 F 1 "VPP" H 1250 3800 50  0000 C CNN
 F 2 "" H 1250 3650 50  0000 C CNN
@@
 PB5
 $Comp
-L +5V #PWR26
+L +5V #PWR026
 U 1 1 58227C48
 P 5200 5650
-F 0 "#PWR26" H 5200 5500 50  0001 C CNN
+F 0 "#PWR026" H 5200 5500 50  0001 C CNN
 F 1 "+5V" H 5200 5790 50  0000 C CNN
 F 2 "" H 5200 5650 50  0000 C CNN
@@
 	3000 4350 3200 4350
 $Comp
-L GND #PWR16
+L GND #PWR027
 U 1 1 585ABDB0
 P 2450 4350
-F 0 "#PWR16" H 2450 4100 50  0001 C CNN
+F 0 "#PWR027" H 2450 4100 50  0001 C CNN
 F 1 "GND" H 2450 4200 50  0000 C CNN
 F 2 "" H 2450 4350 50  0000 C CNN
@@
 	2600 4350 2450 4350
 $Comp
-L +5V #PWR22
-U 1 1 585AC913
-P 4400 2500
-F 0 "#PWR22" H 4400 2350 50  0001 C CNN
-F 1 "+5V" H 4400 2640 50  0000 C CNN
-F 2 "" H 4400 2500 50  0000 C CNN
-F 3 "" H 4400 2500 50  0000 C CNN
-	1    4400 2500
-	1    0    0    -1
-$EndComp
-Wire Wire Line
-	4000 2500 4400 2500
-$Comp
-L +5V #PWR13
+L +5V #PWR028
 U 1 1 585ACDE6
 P 2100 1350
-F 0 "#PWR13" H 2100 1200 50  0001 C CNN
+F 0 "#PWR028" H 2100 1200 50  0001 C CNN
 F 1 "+5V" H 2100 1490 50  0000 C CNN
 F 2 "" H 2100 1350 50  0000 C CNN
@@
 F 0 "IC1" H 2250 3400 50  0000 L BNN
 F 1 "ATMEGA328P-PU" H 3400 750 50  0000 L BNN
-F 2 "DIL28" H 3000 2150 50  0000 C CIN
+F 2 "Housings_DIP:DIP-28_W7.62mm_Socket" H 3000 2150 50  0000 C CIN
 F 3 "" H 3000 2150 50  0000 C CNN
 	1    3000 2150
@@
 F 0 "PB1" H 4750 4700 60  0000 C CNN
 F 1 "push_button" H 5150 4650 60  0001 C CNN
-F 2 "" H 4750 4500 60  0001 C CNN
+F 2 "Buttons_Switches_THT:SW_PUSH-12mm" H 4750 4500 60  0001 C CNN
 F 3 "" H 4750 4500 60  0001 C CNN
 	1    4750 4500
@@
 F 0 "PB2" H 4750 5150 60  0000 C CNN
 F 1 "push_button" H 5150 5100 60  0001 C CNN
-F 2 "" H 4750 4950 60  0001 C CNN
+F 2 "Buttons_Switches_THT:SW_PUSH-12mm" H 4750 4950 60  0001 C CNN
 F 3 "" H 4750 4950 60  0001 C CNN
 	1    4750 4950
@@
 F 0 "D2" H 4750 5750 50  0000 C CNN
 F 1 "LED" H 4750 5550 50  0000 C CNN
-F 2 "" H 4750 5650 50  0000 C CNN
+F 2 "LEDs:LED_D5.0mm" H 4750 5650 50  0001 C CNN
 F 3 "" H 4750 5650 50  0000 C CNN
 	1    4750 5650
@@
 F 0 "SW1" H 4100 5650 60  0000 C CNN
 F 1 "SPST" H 4250 5350 60  0001 C CNN
-F 2 "" H 4250 5550 60  0001 C CNN
+F 2 "Buttons_Switches_THT:SW_Micro_SPST" H 4250 5550 60  0001 C CNN
 F 3 "" H 4250 5550 60  0001 C CNN
 	1    4250 5550
@@
 F 0 "BT1" H 1350 6300 50  0000 L CNN
 F 1 "3V" H 1350 6200 50  0000 L CNN
-F 2 "" V 1250 6260 50  0000 C CNN
+F 2 "custom:CR2032_SMD" V 1250 6260 50  0001 C CNN
 F 3 "" V 1250 6260 50  0000 C CNN
 	1    1250 6200
 	1    0    0    -1
 $EndComp
+$Comp
+L CONN_02X03 P1
+U 1 1 5883BB63
+P 4250 6450
+F 0 "P1" H 4250 6650 50  0000 C CNN
+F 1 "PROGRAMMER" H 4250 6250 50  0000 C CNN
+F 2 "Pin_Headers:Pin_Header_Straight_2x03_Pitch2.54mm" H 4250 5250 50  0001 C CNN
+F 3 "" H 4250 5250 50  0000 C CNN
+	1    4250 6450
+	1    0    0    -1
+$EndComp
+Text GLabel 4000 6350 0    60   Input ~ 0
+PB4
+$Comp
+L +5V #PWR029
+U 1 1 5883EE82
+P 4500 6350
+F 0 "#PWR029" H 4500 6200 50  0001 C CNN
+F 1 "+5V" H 4500 6490 50  0000 C CNN
+F 2 "" H 4500 6350 50  0000 C CNN
+F 3 "" H 4500 6350 50  0000 C CNN
+	1    4500 6350
+	1    0    0    -1
+$EndComp
+Text GLabel 4000 6450 0    60   Input ~ 0
+PB5
+Text GLabel 4500 6450 2    60   Input ~ 0
+PB3
+Text GLabel 4000 2500 2    60   Input ~ 0
+RESET
+Text GLabel 4000 6550 0    60   Input ~ 0
+RESET
+$Comp
+L GND #PWR030
+U 1 1 5883F3CF
+P 4500 6550
+F 0 "#PWR030" H 4500 6300 50  0001 C CNN
+F 1 "GND" H 4500 6400 50  0000 C CNN
+F 2 "" H 4500 6550 50  0000 C CNN
+F 3 "" H 4500 6550 50  0000 C CNN
+	1    4500 6550
+	1    0    0    -1
+$EndComp

Commit message: Re-wire to use hardware PWM d'oh
Changed lines of the file:
@@
 $EndComp
 Text GLabel 1700 3850 1    60   Input ~ 0
-PC3
+PB1
 Text GLabel 5950 4000 3    60   Input ~ 0
 PD5
@@
 PD6
 Text GLabel 6150 1650 1    60   Input ~ 0
-PC0
+PC2
 Text GLabel 5850 1650 1    60   Input ~ 0
-PB3
+PB5
 Text GLabel 5750 1650 1    60   Input ~ 0
-PB2
+PB4
 Text GLabel 5650 4000 3    60   Input ~ 0
 PB0
@@
 PC1
 Text GLabel 6250 1650 1    60   Input ~ 0
-PC1
+PC3
 $Comp
 L GND #PWR09
@@
 $EndComp
 Text GLabel 2800 3750 1    60   Input ~ 0
-PC2
+PB3
 $Comp
 L C_Small C5
@@
 	6050 4000 6050 3750
 Text GLabel 5650 1650 1    60   Input ~ 0
-PB1
+PB2
 Text GLabel 5950 1650 1    60   Input ~ 0
-PB4
+PC0
 Text GLabel 6050 1650 1    60   Input ~ 0
-PB5
+PC1
 Text GLabel 6150 4000 3    60   Input ~ 0
 PD3
@@
 Wire Wire Line
 	3000 4350 3200 4350
-$Comp
-L GND #PWR027
-U 1 1 585ABDB0
-P 2450 4350
-F 0 "#PWR027" H 2450 4100 50  0001 C CNN
-F 1 "GND" H 2450 4200 50  0000 C CNN
-F 2 "" H 2450 4350 50  0000 C CNN
-F 3 "" H 2450 4350 50  0000 C CNN
-	1    2450 4350
-	1    0    0    -1
-$EndComp
 Wire Wire Line
 	2600 4350 2450 4350
 $Comp
-L +5V #PWR028
+L +5V #PWR027
 U 1 1 585ACDE6
 P 2100 1350
-F 0 "#PWR028" H 2100 1200 50  0001 C CNN
+F 0 "#PWR027" H 2100 1200 50  0001 C CNN
 F 1 "+5V" H 2100 1490 50  0000 C CNN
 F 2 "" H 2100 1350 50  0000 C CNN
@@
 PB4
 $Comp
-L +5V #PWR029
+L +5V #PWR028
 U 1 1 5883EE82
 P 4500 6350
-F 0 "#PWR029" H 4500 6200 50  0001 C CNN
+F 0 "#PWR028" H 4500 6200 50  0001 C CNN
 F 1 "+5V" H 4500 6490 50  0000 C CNN
 F 2 "" H 4500 6350 50  0000 C CNN
@@
 RESET
 $Comp
-L GND #PWR030
+L GND #PWR029
 U 1 1 5883F3CF
 P 4500 6550
-F 0 "#PWR030" H 4500 6300 50  0001 C CNN
+F 0 "#PWR029" H 4500 6300 50  0001 C CNN
 F 1 "GND" H 4500 6400 50  0000 C CNN
 F 2 "" H 4500 6550 50  0000 C CNN
@@
 	1    0    0    -1
 $EndComp
+$Comp
+L +5V #PWR030
+U 1 1 58C89AC3
+P 2450 4350
+F 0 "#PWR030" H 2450 4200 50  0001 C CNN
+F 1 "+5V" H 2450 4490 50  0000 C CNN
+F 2 "" H 2450 4350 50  0000 C CNN
+F 3 "" H 2450 4350 50  0000 C CNN
+	1    2450 4350
+	1    0    0    -1
+$EndComp
