File: hardware/alarm-clock.sch (KiCad schematic (older format))
At the start: 36 parts, among them CON1 BARREL_JACK, CON2 BARREL_JACK, IC1 ATMEGA328P-PU, P1 PROGRAMMER, Q1 Q_NPN_BCE, Q2 Q_NPN_BCE, SW1 SPST, U1 LM7805CT, U2 DS1307, U3 4Dig7Seg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

Commit message: WIP V3
Parts:
- removed IC1: ATMEGA328P-PU, Housings_DIP:DIP-28_W7.62mm_Socket, symbol ATMEGA328P-PU
- removed R10, R11, R12, R13, R14, R3, R6, R7, R8, R9: 2.2k, Resistors_SMD:R_1210_HandSoldering, symbol R
- removed U2: DS1307, Housings_DIP:DIP-8_W7.62mm_LongPads, symbol DS1307
- removed U3: 4Dig7Seg, custom:4Dig7Seg, symbol 4Dig7Seg
- removed Y1: 38.7kHz, Crystals:Crystal_Round_Horizontal_2mm, symbol Crystal_Small
- added J1: CONN_01X04, Pin_Headers:Pin_Header_Straight_1x04_Pitch2.54mm, symbol CONN_01X04
- added PB2: push_button, custom:KS_BUTTON, symbol push_button
- added R5: 2k2, Resistors_SMD:R_1206_HandSoldering, symbol R
- added U2: DS3232, Housings_SOIC:SOIC-20W_7.5x12.8mm_Pitch1.27mm, symbol DS3232-RESCUE-alarm-clock
- added U3: ATMEGA328-AU, Housings_QFP:TQFP-32_7x7mm_Pitch0.8mm, symbol ATMEGA328-AU
- C1: footprint Capacitors_ThroughHole:C_Radial_D6.3_L11.2_P2.5 -> Capacitors_SMD:C_1206_HandSoldering
- C2: renamed from C3; footprint Capacitors_ThroughHole:C_Radial_D5_L11_P2 -> Capacitors_SMD:C_1206_HandSoldering
- C3: renamed from C5; footprint Capacitors_ThroughHole:C_Disc_D3_P2.5 -> Capacitors_SMD:C_1206_HandSoldering
- C4: renamed from C6; footprint Capacitors_ThroughHole:C_Disc_D3_P2.5 -> Capacitors_SMD:C_1206_HandSoldering
- D1: footprint Diodes_THT:Diode_DO-41_SOD81_Horizontal_RM10 -> Diodes_SMD:D_1206
- D2: footprint LEDs:LED_D5.0mm -> LEDs:LED_1206
- PB1: footprint Buttons_Switches_THT:SW_PUSH-12mm -> custom:KS_BUTTON
- PB3: renamed from PB2; footprint Buttons_Switches_THT:SW_PUSH-12mm -> custom:KS_BUTTON
- R1, R2: value 3.3k -> 3k3; footprint Resistors_SMD:R_1210_HandSoldering -> Resistors_SMD:R_1206_HandSoldering
- R3: renamed from R5; value 270 -> 2k2; footprint Resistors_SMD:R_1210_HandSoldering -> Resistors_SMD:R_1206_HandSoldering
- R4: value 2.2k -> 2k2; footprint Resistors_SMD:R_1210_HandSoldering -> Resistors_SMD:R_1206_HandSoldering
- U1: footprint Power_Integrations:TO-220 -> TO_SOT_Packages_THT:TO-220_Horizontal
- renumbered Y2 to Y1
Connections:
- net labels added: SCL, SDA
- net labels removed: PC4, PC5
- wire segments 57 -> 47
- no-connect marks 2 -> 4
